Commit message: add gazebo sensors and launch for tf_wrapper/relay

File: ros_robotics/src/description/urdf/robot.urdf.xacro (robot description, xacro)
@@ -77,5 +77,4 @@
         </geometry>
     </xacro:macro>
-    <link name="dummy_link"></link>
     <!-- Корпус робота -->
     <link name="base_link">
@@ -90,9 +89,4 @@
         </collision>
     </link>
-    <joint name="dummy_joint" type="fixed">
-        <origin rpy="0 0 0" xyz="0 0 0" />
-        <parent link="dummy_link"/>
-        <child link="base_link"/>
-	</joint>
     <!-- Усовершенствованный макрос для создания ноги -->
     <xacro:macro name="leg" params="prefix length1 length2 reflect_x reflect_y">
@@ -149,4 +143,11 @@
             </collision>
         </link>
+        <!-- Датчик силы на стопе -->
+        <link name="${prefix}_foot_force_sensor_link">
+            <inertial>
+                <mass value="0.001"/>  <!-- Минимальная масса -->
+                <inertia ixx="0.00001" ixy="0.0" ixz="0.0" iyy="0.00001" iyz="0.0" izz="0.00001"/>
+            </inertial>
+        </link>
         <!-- Соединение первого сегмента с корпусом -->
         <joint name="${prefix}_leg1_corpus_joint" type="revolute">
@@ -173,4 +174,9 @@
             <origin xyz="0 0 ${-length2}" rpy="0 0 0"/>
         </joint>
+        <joint name="${prefix}_foot_force_sensor_joint" type="fixed">
+            <parent link="${prefix}_foot_link"/>  <!-- Родительское звено стопы -->
+            <child link="${prefix}_foot_force_sensor_link"/>
+            <origin xyz="0 0 -0.05" rpy="0 0 0"/>  <!-- Размещение под стопой -->
+        </joint>
     </xacro:macro>
     <!-- Создание всех четырех ног -->

File: ros_robotics/src/description/urdf/robot_gazebo.urdf.xacro (robot description, xacro)
@@ -30,4 +30,20 @@
             <kd>1000</kd> <!-- Демпфирование -->
         </gazebo>
+        <!-- Gazebo plugin для измерения силы -->
+        <gazebo reference="${prefix}_foot_force_sensor_link">
+            <sensor name="${prefix}_foot_force_sensor" type="force_torque">
+                <always_on>true</always_on>
+                <update_rate>100</update_rate>
+                <plugin filename="libgazebo_ros_ft_sensor.so" name="ft_sensor_plugin">
+                    <topic_name>/sensors/force/${prefix}_foot</topic_name>
+                    <frame_name>${prefix}_foot_force_sensor_link</frame_name>
+                    <noise>
+                        <type>gaussian</type>
+                        <mean>0.0</mean>
+                        <stddev>0.1</stddev>  <!-- Уровень шума -->
+                    </noise>
+                </plugin>
+            </sensor>
+        </gazebo>
     </xacro:macro>
     <xacro:leg_color_gazebo prefix="front_right"/>
@@ -35,4 +51,24 @@
     <xacro:leg_color_gazebo prefix="front_left"/>
     <xacro:leg_color_gazebo prefix="back_left"/>
+    <gazebo reference="base_link">
+        <gravity>true</gravity>
+        <sensor name="imu_sensor" type="imu">
+            <always_on>true</always_on>
+            <update_rate>100</update_rate>
+            <visualize>true</visualize>
+            <topic>__default_topic__</topic>
+            <plugin filename="libgazebo_ros_imu_sensor.so" name="imu_plugin">
+                <topicName>imu/data_raw</topicName>
+                <bodyName>base_link</bodyName>
+                <updateRateHZ>10.0</updateRateHZ>
+                <gaussianNoise>0.005</gaussianNoise>
+                <xyzOffset>0 0 0</xyzOffset>
+                <rpyOffset>0 0 0</rpyOffset>
+                <frameName>base_link</frameName>
+                <initialOrientationAsReference>false</initialOrientationAsReference>
+            </plugin>
+            <pose>0 0 0 0 0 0</pose>
+        </sensor>
+    </gazebo>
     <gazebo>
         <plugin filename="libgazebo_ros2_control.so" name="gazebo_ros2_control">

File: ros_robotics/src/description/urdf/robot_ros.urdf.xacro (robot description, xacro)
@@ -6,34 +6,42 @@
         </hardware>
         <joint name="front_right_leg1_corpus_joint">
-            <command_interface name="position" />
+            <command_interface name="effort" />
             <state_interface name="position"/>
+            <state_interface name="velocity"/>
         </joint>
         <joint name="back_right_leg1_corpus_joint">
-            <command_interface name="position" />
+            <command_interface name="effort" />
             <state_interface name="position"/>
+            <state_interface name="velocity"/>
         </joint>
         <joint name="front_left_leg1_corpus_joint">
-            <command_interface name="position" />
+            <command_interface name="effort" />
             <state_interface name="position"/>
+            <state_interface name="velocity"/>
         </joint>
         <joint name="back_left_leg1_corpus_joint">
-            <command_interface name="position" />
+            <command_interface name="effort" />
             <state_interface name="position"/>
+            <state_interface name="velocity"/>
         </joint>
         <joint name="front_right_leg1_leg2_joint">
-            <command_interface name="position" />
+            <command_interface name="effort" />
             <state_interface name="position"/>
+            <state_interface name="velocity"/>
         </joint>
         <joint name="back_right_leg1_leg2_joint">
-            <command_interface name="position" />
+            <command_interface name="effort" />
             <state_interface name="position"/>
+            <state_interface name="velocity"/>
         </joint>
         <joint name="front_left_leg1_leg2_joint">
-            <command_interface name="position" />
+            <command_interface name="effort" />
             <state_interface name="position"/>
+            <state_interface name="velocity"/>
         </joint>
         <joint name="back_left_leg1_leg2_joint">
-            <command_interface name="position" />
+            <command_interface name="effort" />
             <state_interface name="position"/>
+            <state_interface name="velocity"/>
         </joint>
     </ros2_control>

Commit message: add inverse_kinematics to stand_up_node

File: ros_robotics/src/description/urdf/robot.urdf.xacro (robot description, xacro)
@@ -154,7 +154,7 @@
             <parent link="base_link"/>
             <child link="${prefix}_leg1_link"/>
-            <origin xyz="${reflect_x * corpus_width/2} ${reflect_y * (corpus_length/2 - leg1_shift_y)} ${leg1_shift_z}" rpy="${leg1_angle_x} 0 0"/>
+            <origin xyz="${reflect_x * corpus_width/2} ${reflect_y * (corpus_length/2 - leg1_shift_y)} ${leg1_shift_z}" rpy="${-leg1_angle_x} 0 0"/>
             <axis xyz="1 0 0"/>
-            <limit effort="150.0" lower="${leg1_angle_x}" upper="${-leg1_angle_x}" velocity="3.0"/>
+            <limit effort="150.0" lower="${leg1_angle_lower_x}" upper="${leg1_angle_upper_x}" velocity="3.0"/>
             <dynamics damping="0.7" friction="0.1"/>
         </joint>
@@ -165,5 +165,5 @@
             <origin xyz="0 0 ${-length1}" rpy="${leg2_angle_x} 0 0"/>
             <axis xyz="1 0 0"/>
-            <limit effort="120.0" lower="${-leg2_angle_x}" upper="${PI/12}" velocity="4.0"/>
+            <limit effort="120.0" lower="${leg2_angle_lower_x}" upper="${leg2_angle_upper_x}" velocity="4.0"/>
             <dynamics damping="0.5" friction="0.1"/>
         </joint>

File: ros_robotics/src/description/urdf/robot_property.urdf.xacro (robot description, xacro)
@@ -26,6 +26,10 @@
     <xacro:property name="leg1_shift_y" value="${corpus_length/10}" />
     <xacro:property name="leg1_shift_z" value="${corpus_height/4}" />
-    <xacro:property name="leg1_angle_x" value="${-PI/4}" />
+    <xacro:property name="leg1_angle_x" value="${PI/4}" />
+    <xacro:property name="leg1_angle_lower_x" value="${-PI/4}" />
+    <xacro:property name="leg1_angle_upper_x" value="${PI/4}" />
     <!-- Параметры для второго сегмента ноги -->
     <xacro:property name="leg2_angle_x" value="${PI/2}" />
+    <xacro:property name="leg2_angle_lower_x" value="${leg1_angle_lower_x}" />
+    <xacro:property name="leg2_angle_upper_x" value="${PI/12}" />
 </robot>
